Commit message: add mini_cheetah vis

File: robots/xpp_arcdog/urdf/mini_cheetah.urdf.xacro (robot description, xacro)
@@ -4,5 +4,18 @@
         <color rgba=".2 .2 .2 1"/>
     </material>
-    <link name="body">
+    <link name="base">
+      <visual>
+        <origin rpy="0 0 0" xyz="0 0 0"/>
+        <geometry>
+          <box size="0.001 0.001 0.001"/>
+        </geometry>
+      </visual>
+    </link>
+    <joint name="floating_base" type="fixed">
+      <origin rpy="0 0 0" xyz="0 0 0"/>
+      <parent link="base"/>
+      <child link="trunk"/>
+    </joint>
+    <link name="trunk">
         <inertial>
             <mass value="3.3"/>
@@ -24,11 +37,11 @@
     </link>
     <!--!!!!!!!!!!!! Front Right Leg !!!!!!!!!!!!!!!!!!!!!!!!!!!!!!!!!!!!-->
-    <joint name="torso_to_abduct_fr_j" type="continuous">
+    <joint name="FR_hip_joint" type="continuous">
         <axis xyz="1 0 0"/>
         <origin rpy="0 0 0" xyz="0.19 -0.049 0.0"/>
-        <parent link="body"/>
-        <child link="abduct_fr"/>
-    </joint>
-    <link name="abduct_fr">
+        <parent link="trunk"/>
+        <child link="FR_hip"/>
+    </joint>
+    <link name="FR_hip">
         <inertial>
             <mass value="0.54"/>
@@ -50,11 +63,11 @@
         </collision>
     </link>
-    <joint name="abduct_fr_to_thigh_fr_j" type="continuous">
+    <joint name="FR_thigh_joint" type="continuous">
         <axis xyz="0 -1 0"/>
         <origin rpy="0.0 0.0 0.0" xyz="0.0 -0.062 0.00"/>
-        <parent link="abduct_fr"/>
-        <child link="thigh_fr"/>
-    </joint>
-    <link name="thigh_fr">
+        <parent link="FR_hip"/>
+        <child link="FR_thigh"/>
+    </joint>
+    <link name="FR_thigh">
         <inertial>
             <mass value="0.634"/>
@@ -76,11 +89,11 @@
         </collision>
     </link>
-    <joint name="thigh_fr_to_knee_fr_j" type="continuous">
+    <joint name="FR_calf_joint" type="continuous">
         <axis xyz="0 -1 0"/>
         <origin rpy="0.0 0 0.0" xyz="0.0 0.0 -0.209"/>
-        <parent link="thigh_fr"/>
-        <child link="shank_fr"/>
-    </joint>
-    <link name="shank_fr">
+        <parent link="FR_thigh"/>
+        <child link="FR_calf"/>
+    </joint>
+    <link name="FR_calf">
         <inertial>
             <mass value="0.064"/>
@@ -128,5 +141,5 @@
   </link>
   <joint name="toe_fr_joint" type="fixed">
-    <parent link="shank_fr"/>
+    <parent link="FR_calf"/>
     <child link="toe_fr"/>
     <origin xyz="0 0 -0.18"/>
@@ -134,11 +147,11 @@
   </joint>
 <!--!!!!!!!!!!!! Front Left Leg !!!!!!!!!!!!!!!!!!!!!!!!!!!!!!!!!!!!-->
-    <joint name="torso_to_abduct_fl_j" type="continuous">
+    <joint name="FL_hip_joint" type="continuous">
         <axis xyz="1 0 0"/>
         <origin rpy="0 0 0" xyz="0.19 0.049 0.0"/>
-        <parent link="body"/>
-        <child link="abduct_fl"/>
-    </joint>
-    <link name="abduct_fl">
+        <parent link="trunk"/>
+        <child link="FL_hip"/>
+    </joint>
+    <link name="FL_hip">
         <inertial>
             <mass value="0.54"/>
@@ -160,11 +173,11 @@
         </collision>
     </link>
-    <joint name="abduct_fl_to_thigh_fl_j" type="continuous">
+    <joint name="FL_thigh_joint" type="continuous">
         <axis xyz="0 -1 0"/>
         <origin rpy="0.0 0.0 0.0" xyz="0.0 0.062 0.00"/>
-        <parent link="abduct_fl"/>
-        <child link="thigh_fl"/>
-    </joint>
-    <link name="thigh_fl">
+        <parent link="FL_hip"/>
+        <child link="FL_thigh"/>
+    </joint>
+    <link name="FL_thigh">
         <inertial>
             <mass value="0.634"/>
@@ -186,11 +199,11 @@
         </collision>
     </link>
-    <joint name="thigh_fl_to_knee_fl_j" type="continuous">
+    <joint name="FL_calf_joint" type="continuous">
         <axis xyz="0 -1 0"/>
         <origin rpy="0.0 0 0.0" xyz="0.0 0.0 -0.209"/>
-        <parent link="thigh_fl"/>
-        <child link="shank_fl"/>
-    </joint>
-    <link name="shank_fl">
+        <parent link="FL_thigh"/>
+        <child link="FL_calf"/>
+    </joint>
+    <link name="FL_calf">
         <inertial>
             <mass value="0.064"/>
@@ -238,5 +251,5 @@
   </link>
   <joint name="toe_fl_joint" type="fixed">
-    <parent link="shank_fl"/>
+    <parent link="FL_calf"/>
     <child link="toe_fl"/>
     <origin xyz="0 0 -0.18"/>
@@ -244,11 +257,11 @@
   </joint>
 <!--!!!!!!!!!!!! Hind Right Leg !!!!!!!!!!!!!!!!!!!!!!!!!!!!!!!!!!!!-->
-    <joint name="torso_to_abduct_hr_j" type="continuous">
+    <joint name="RR_hip_joint" type="continuous">
         <axis xyz="1 0 0"/>
         <origin rpy="0 0 0" xyz="-0.19 -0.049 0.0"/>
-        <parent link="body"/>
-        <child link="abduct_hr"/>
-    </joint>
-    <link name="abduct_hr">
+        <parent link="trunk"/>
+        <child link="RR_hip"/>
+    </joint>
+    <link name="RR_hip">
         <inertial>
             <mass value="0.54"/>
@@ -270,11 +283,11 @@
         </collision>
     </link>
-    <joint name="abduct_hr_to_thigh_hr_j" type="continuous">
+    <joint name="RR_thigh_joint" type="continuous">
         <axis xyz="0 -1 0"/>
         <origin rpy="0.0 0.0 0.0" xyz="0.0 -0.062 0.00"/>
-        <parent link="abduct_hr"/>
-        <child link="thigh_hr"/>
-    </joint>
-    <link name="thigh_hr">
+        <parent link="RR_hip"/>
+        <child link="RR_thigh"/>
+    </joint>
+    <link name="RR_thigh">
         <inertial>
             <mass value="0.634"/>
@@ -296,11 +309,11 @@
         </collision>
     </link>
-    <joint name="thigh_hr_to_knee_hr_j" type="continuous">
+    <joint name="RR_calf_joint" type="continuous">
         <axis xyz="0 -1 0"/>
         <origin rpy="0.0 0 0.0" xyz="0.0 0.0 -0.209"/>
-        <parent link="thigh_hr"/>
-        <child link="shank_hr"/>
-    </joint>
-    <link name="shank_hr">
+        <parent link="RR_thigh"/>
+        <child link="RR_calf"/>
+    </joint>
+    <link name="RR_calf">
         <inertial>
             <mass value="0.064"/>
@@ -348,5 +361,5 @@
   </link>
   <joint name="toe_hr_joint" type="fixed">
-    <parent link="shank_hr"/>
+    <parent link="RR_calf"/>
     <child link="toe_hr"/>
     <origin xyz="0 0 -0.18"/>
@@ -354,11 +367,11 @@
   </joint>
 <!--!!!!!!!!!!!! Hind Left Leg !!!!!!!!!!!!!!!!!!!!!!!!!!!!!!!!!!!!-->
-    <joint name="torso_to_abduct_hl_j" type="continuous">
+    <joint name="RL_hip_joint" type="continuous">
         <axis xyz="1 0 0"/>
         <origin rpy="0 0 0" xyz="-0.19 0.049 0.0"/>
-        <parent link="body"/>
-        <child link="abduct_hl"/>
-    </joint>
-    <link name="abduct_hl">
+        <parent link="trunk"/>
+        <child link="RL_hip"/>
+    </joint>
+    <link name="RL_hip">
         <inertial>
             <mass value="0.54"/>
@@ -380,11 +393,11 @@
         </collision>
     </link>
-    <joint name="abduct_hl_to_thigh_hl_j" type="continuous">
+    <joint name="RL_thigh_joint" type="continuous">
         <axis xyz="0 -1 0"/>
         <origin rpy="0.0 0.0 0.0" xyz="0.0 0.062 0.00"/>
-        <parent link="abduct_hl"/>
-        <child link="thigh_hl"/>
-    </joint>
-    <link name="thigh_hl">
+        <parent link="RL_hip"/>
+        <child link="RL_thigh"/>
+    </joint>
+    <link name="RL_thigh">
         <inertial>
             <mass value="0.634"/>
@@ -406,11 +419,11 @@
         </collision>
     </link>
-    <joint name="thigh_hl_to_knee_hl_j" type="continuous">
+    <joint name="RL_calf_joint" type="continuous">
         <axis xyz="0 -1 0"/>
         <origin rpy="0.0 0 0.0" xyz="0.0 0.0 -0.209"/>
-        <parent link="thigh_hl"/>
-        <child link="shank_hl"/>
-    </joint>
-    <link name="shank_hl">
+        <parent link="RL_thigh"/>
+        <child link="RL_calf"/>
+    </joint>
+    <link name="RL_calf">
         <inertial>
             <mass value="0.064"/>
@@ -458,5 +471,5 @@
   </link>
   <joint name="toe_hl_joint" type="fixed">
-    <parent link="shank_hl"/>
+    <parent link="RL_calf"/>
     <child link="toe_hl"/>
     <origin xyz="0 0 -0.18"/>

Commit message: fix revolute joint direction

File: robots/xpp_arcdog/urdf/mini_cheetah.urdf.xacro (robot description, xacro)
@@ -42,4 +42,12 @@
         <parent link="trunk"/>
         <child link="FR_hip"/>
+        <limit
+        lower="-0.75"
+        upper="0.75"
+        effort="17"
+        velocity="12" />
+        <dynamics
+        damping="0.01"
+        friction="0.2" />
     </joint>
     <link name="FR_hip">
@@ -64,8 +72,16 @@
     </link>
     <joint name="FR_thigh_joint" type="continuous">
-        <axis xyz="0 -1 0"/>
+        <axis xyz="0 1 0"/>
         <origin rpy="0.0 0.0 0.0" xyz="0.0 -0.062 0.00"/>
         <parent link="FR_hip"/>
         <child link="FR_thigh"/>
+        <limit
+         lower="-1.257"
+         upper="4.363"
+         effort="24"
+         velocity="12" />
+        <dynamics
+         damping="0.01"
+         friction="0.2" />
     </joint>
     <link name="FR_thigh">
@@ -90,8 +106,16 @@
     </link>
     <joint name="FR_calf_joint" type="continuous">
-        <axis xyz="0 -1 0"/>
+        <axis xyz="0 1 0"/>
         <origin rpy="0.0 0 0.0" xyz="0.0 0.0 -0.209"/>
         <parent link="FR_thigh"/>
         <child link="FR_calf"/>
+        <limit
+          lower="-2.478"
+          upper="-0.506"
+          effort="24"
+          velocity="12" />
+        <dynamics
+          damping="0.01"
+          friction="0.2" />
     </joint>
     <link name="FR_calf">
@@ -152,4 +176,12 @@
         <parent link="trunk"/>
         <child link="FL_hip"/>
+        <limit
+        lower="-0.75"
+        upper="0.75"
+        effort="17"
+        velocity="12" />
+        <dynamics
+        damping="0.01"
+        friction="0.2" />
     </joint>
     <link name="FL_hip">
@@ -174,8 +206,16 @@
     </link>
     <joint name="FL_thigh_joint" type="continuous">
-        <axis xyz="0 -1 0"/>
+        <axis xyz="0 1 0"/>
         <origin rpy="0.0 0.0 0.0" xyz="0.0 0.062 0.00"/>
         <parent link="FL_hip"/>
         <child link="FL_thigh"/>
+        <limit
+          lower="-1.257"
+          upper="4.363"
+          effort="24"
+          velocity="12" />
+        <dynamics
+          damping="0.01"
+          friction="0.2" />
     </joint>
     <link name="FL_thigh">
@@ -200,8 +240,16 @@
     </link>
     <joint name="FL_calf_joint" type="continuous">
-        <axis xyz="0 -1 0"/>
+        <axis xyz="0 1 0"/>
         <origin rpy="0.0 0 0.0" xyz="0.0 0.0 -0.209"/>
         <parent link="FL_thigh"/>
         <child link="FL_calf"/>
+        <limit
+          lower="-2.478"
+          upper="-0.506"
+          effort="24"
+          velocity="12" />
+        <dynamics
+          damping="0.01"
+          friction="0.2" />
     </joint>
     <link name="FL_calf">
@@ -262,4 +310,12 @@
         <parent link="trunk"/>
         <child link="RR_hip"/>
+        <limit
+          lower="-0.75"
+          upper="0.75"
+          effort="17"
+          velocity="12" />
+        <dynamics
+          damping="0.01"
+          friction="0.2" />
     </joint>
     <link name="RR_hip">
@@ -284,8 +340,16 @@
     </link>
     <joint name="RR_thigh_joint" type="continuous">
-        <axis xyz="0 -1 0"/>
+        <axis xyz="0 1 0"/>
         <origin rpy="0.0 0.0 0.0" xyz="0.0 -0.062 0.00"/>
         <parent link="RR_hip"/>
         <child link="RR_thigh"/>
+        <limit
+          lower="-2.01"
+          upper="3.49"
+          effort="24"
+          velocity="12" />
+        <dynamics
+          damping="0.01"
+          friction="0.2" />
     </joint>
     <link name="RR_thigh">
@@ -310,8 +374,16 @@
     </link>
     <joint name="RR_calf_joint" type="continuous">
-        <axis xyz="0 -1 0"/>
+        <axis xyz="0 1 0"/>
         <origin rpy="0.0 0 0.0" xyz="0.0 0.0 -0.209"/>
         <parent link="RR_thigh"/>
         <child link="RR_calf"/>
+        <limit
+          lower="-2.478"
+          upper="-0.506"
+          effort="24"
+          velocity="12" />
+        <dynamics
+          damping="0.01"
+          friction="0.2" />
     </joint>
     <link name="RR_calf">
@@ -372,4 +444,12 @@
         <parent link="trunk"/>
         <child link="RL_hip"/>
+        <limit
+          lower="-0.75"
+          upper="0.75"
+          effort="17"
+          velocity="12" />
+        <dynamics
+          damping="0.01"
+          friction="0.2" />
     </joint>
     <link name="RL_hip">
@@ -394,8 +474,16 @@
     </link>
     <joint name="RL_thigh_joint" type="continuous">
-        <axis xyz="0 -1 0"/>
+        <axis xyz="0 1 0"/>
         <origin rpy="0.0 0.0 0.0" xyz="0.0 0.062 0.00"/>
         <parent link="RL_hip"/>
         <child link="RL_thigh"/>
+        <limit
+          lower="-2.01"
+          upper="3.49"
+          effort="24"
+          velocity="12" />
+        <dynamics
+          damping="0.01"
+          friction="0.2" />
     </joint>
     <link name="RL_thigh">
@@ -420,8 +508,16 @@
     </link>
     <joint name="RL_calf_joint" type="continuous">
-        <axis xyz="0 -1 0"/>
+        <axis xyz="0 1 0"/>
         <origin rpy="0.0 0 0.0" xyz="0.0 0.0 -0.209"/>
         <parent link="RL_thigh"/>
         <child link="RL_calf"/>
+        <limit
+          lower="-2.478"
+          upper="-0.506"
+          effort="24"
+          velocity="12" />
+        <dynamics
+          damping="0.01"
+          friction="0.2" />
     </joint>
     <link name="RL_calf">
