Commit message: new arcdog model

File: robots/xpp_arcdog/urdf/arcdog.urdf.xacro (robot description, xacro)
@@ -73,5 +73,5 @@
     <joint name="FR_thigh_joint" type="continuous">
         <axis xyz="0 1 0"/>
-        <origin rpy="0.0 0.0 0.0" xyz="0.0 -0.0972 0.00"/>
+        <origin rpy="0.0 0.0 0.0" xyz="0.0 -0.1165 0.00"/>
         <parent link="FR_hip"/>
         <child link="FR_thigh"/>
@@ -167,5 +167,5 @@
     <parent link="FR_calf"/>
     <child link="toe_fr"/>
-    <origin xyz="0 0 -0.2485"/>
+    <origin xyz="0 0 -0.23704"/>
     <dynamics damping="0.0" friction="0.0"/>
   </joint>
@@ -207,5 +207,5 @@
     <joint name="FL_thigh_joint" type="continuous">
         <axis xyz="0 1 0"/>
-        <origin rpy="0.0 0.0 0.0" xyz="0.0 0.0972 0.00"/>
+        <origin rpy="0.0 0.0 0.0" xyz="0.0 0.1165 0.00"/>
         <parent link="FL_hip"/>
         <child link="FL_thigh"/>
@@ -301,5 +301,5 @@
     <parent link="FL_calf"/>
     <child link="toe_fl"/>
-    <origin xyz="0 0 -0.2485"/>
+    <origin xyz="0 0 -0.23704"/>
     <dynamics damping="0.0" friction="0.0"/>
   </joint>
@@ -341,5 +341,5 @@
     <joint name="RR_thigh_joint" type="continuous">
         <axis xyz="0 1 0"/>
-        <origin rpy="0.0 0.0 0.0" xyz="0.0 -0.0972 0.00"/>
+        <origin rpy="0.0 0.0 0.0" xyz="0.0 -0.1165 0.00"/>
         <parent link="RR_hip"/>
         <child link="RR_thigh"/>
@@ -435,5 +435,5 @@
     <parent link="RR_calf"/>
     <child link="toe_hr"/>
-    <origin xyz="0 0 -0.2485"/>
+    <origin xyz="0 0 -0.23704"/>
     <dynamics damping="0.0" friction="0.0"/>
   </joint>
@@ -475,5 +475,5 @@
     <joint name="RL_thigh_joint" type="continuous">
         <axis xyz="0 1 0"/>
-        <origin rpy="0.0 0.0 0.0" xyz="0.0 0.0972 0.00"/>
+        <origin rpy="0.0 0.0 0.0" xyz="0.0 0.1165 0.00"/>
         <parent link="RL_hip"/>
         <child link="RL_thigh"/>
@@ -569,5 +569,5 @@
     <parent link="RL_calf"/>
     <child link="toe_hl"/>
-    <origin xyz="0 0 -0.2485"/>
+    <origin xyz="0 0 -0.23704"/>
     <dynamics damping="0.0" friction="0.0"/>
   </joint>
